File: tests/line-follower/schematics/line-detector/_autosave-line-detector.kicad_sch (KiCad schematic)
At the start: 11 parts, among them J1 ir_module1, J2 ir_module2, J3 ouput_to_mcu, U1 LM339

Commit message: added ir couplet
Parts:
- gave numbers to parts that had none: 1
Changed lines of the file:
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@@
   (symbol (lib_id "Comparator:LM339") (at 146.05 62.23 0) (unit 5)
     (in_bom yes) (on_board yes) (fields_autoplaced)
-    (property "Reference" "U?" (id 0) (at 144.78 60.9599 0)
+    (property "Reference" "U2" (id 0) (at 144.78 60.9599 0)
       (effects (font (size 1.27 1.27)) (justify left))
     )
@@
   (symbol (lib_id "power:GND") (at 143.51 69.85 0) (unit 1)
     (in_bom yes) (on_board yes) (fields_autoplaced)
-    (property "Reference" "#PWR?" (id 0) (at 143.51 76.2 0)
+    (property "Reference" "#PWR0101" (id 0) (at 143.51 76.2 0)
       (effects (font (size 1.27 1.27)) hide)
     )
@@
     )
     (path "/dc446d3f-bb1e-4ad8-94ec-be870693c0f3"
-      (reference "#PWR?") (unit 1) (value "GND") (footprint "")
+      (reference "#PWR0101") (unit 1) (value "GND") (footprint "")
     )
     (path "/2c966f40-766d-457c-9d3a-710432323578"
@@
     )
     (path "/d3d53759-53c2-459c-9fbe-fdde3d5b71e2"
-      (reference "U?") (unit 5) (value "LM339") (footprint "")
+      (reference "U2") (unit 5) (value "LM339") (footprint "")
     )
   )
